File: hw-hand386/PicoGUS.kicad_pcb (KiCad board)
At the start: 4 copper layers, 29.2 x 75.2 mm, 45 parts, among them J1 AudioJack3, J3 Bus_ISA_8bit, J5 PJ-208-SMD, J6 UART_TX, U1 Pico, U10 PCM5100, U2 74LVC244, U3 SN74CB3T3257, U4 SN74CB3T3257, U5 74LVC14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

Commit message: Tweaks
Parts:
- FB1: renamed from L1; footprint Inductor_SMD:L_0402_1005Metric -> Inductor_SMD:L_0603_1608Metric
- FB2: renamed from L2; footprint Inductor_SMD:L_0402_1005Metric -> Inductor_SMD:L_0603_1608Metric
- J5: value PJ-208-SMD -> AudioJack3
- U2: value 74LVC244 -> SN74CB3T3245
- moved R3 1.92 mm to (128.4, 62.7)
- moved R4 1.91 mm to (128.4, 60.7)
- moved FB1 0.90 mm to (131.7, 62.9), turned to 0 degrees
- moved FB2 0.90 mm to (131.7, 60.8), turned to 0 degrees
- moved U7 0.59 mm to (137.8, 74.2)
- moved C20 0.13 mm to (140.6, 73.7)
Routing:
- net GND: track 56.7 -> 73.5 mm, vias 50 -> 75
- net +3V3: track 32.9 -> 38.1 mm, vias 26 -> 36
- net +5V: track 76.0 -> 78.0 mm, vias 5 -> 8
- net Net-(U6-Pad10): track 17.9 -> 16.8 mm
- net A0: track 29.8 -> 28.8 mm
- net AEN: track 34.3 -> 33.7 mm
- net DACK: track 41.6 -> 41.1 mm
