File: hw-hand386/PicoGUS.kicad_sch (KiCad schematic)
At the start: 33 parts, among them J1 AudioJack3, J3 Bus_ISA_8bit, J5 SJ1-3535NG, J6 UART_TX, U1 Pico, U2 74LVC244, U3 SN74CB3T3257, U4 SN74CB3T3257, U5 74LVC14, U6 74LVC00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

Commit message: Tweaks
Parts:
- FB1: renamed from L1; footprint Inductor_SMD:L_0402_1005Metric -> Inductor_SMD:L_0603_1608Metric
- FB2: renamed from L2; footprint Inductor_SMD:L_0402_1005Metric -> Inductor_SMD:L_0603_1608Metric
- J5: value SJ1-3535NG -> AudioJack3
- U2: value 74LVC244 -> SN74CB3T3245
Changed lines of the file:
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@@
   )
   (symbol (lib_id "Connector:Bus_ISA_8bit") (at 46.355 62.23 0) (unit 1)
-    (in_bom yes) (on_board yes) (dnp no)
+    (in_bom yes) (on_board no) (dnp no)
     (property "Reference" "J3" (at 45.72 13.97 0)
       (effects (font (size 1.27 1.27)))
@@
   (symbol (lib_id "Connector_Audio:AudioJack3") (at 252.73 49.53 180) (unit 1)
     (in_bom yes) (on_board yes) (dnp no) (fields_autoplaced)
-    (property "Reference" "J5" (at 260.35 45.0849 0)
+    (property "Reference" "J5" (at 260.35 47.625 0)
       (effects (font (size 1.27 1.27)) (justify right))
     )
-    (property "Value" "SJ1-3535NG" (at 260.35 47.6249 0)
+    (property "Value" "AudioJack3" (at 260.35 50.165 0)
       (effects (font (size 1.27 1.27)) (justify right))
     )
@@
   (symbol (lib_id "74xx:74HC244") (at 132.715 131.445 0) (unit 1)
     (in_bom yes) (on_board yes) (dnp no) (fields_autoplaced)
-    (property "Reference" "U2" (at 134.7344 110.49 0)
-      (effects (font (size 1.27 1.27)) (justify left))
-    )
-    (property "Value" "74LVC244" (at 134.7344 113.03 0)
+    (property "Reference" "U2" (at 134.6709 111.76 0)
+      (effects (font (size 1.27 1.27)) (justify left))
+    )
+    (property "Value" "SN74CB3T3245" (at 134.6709 114.3 0)
       (effects (font (size 1.27 1.27)) (justify left))
     )
@@
   )
   (symbol (lib_id "PiGUS library:Pico") (at 109.22 61.595 0) (unit 1)
-    (in_bom yes) (on_board yes) (dnp no) (fields_autoplaced)
+    (in_bom yes) (on_board no) (dnp no) (fields_autoplaced)
     (property "Reference" "U1" (at 109.22 29.845 0)
       (effects (font (size 1.27 1.27)))
@@
   (symbol (lib_id "Device:FerriteBead") (at 224.79 54.61 90) (unit 1)
     (in_bom yes) (on_board yes) (dnp no)
-    (property "Reference" "L1" (at 227.33 48.26 90)
+    (property "Reference" "FB1" (at 227.33 48.26 90)
       (effects (font (size 1.27 1.27)))
     )
@@
       (effects (font (size 1.27 1.27)))
     )
-    (property "Footprint" "Inductor_SMD:L_0402_1005Metric" (at 224.79 56.388 90)
+    (property "Footprint" "Inductor_SMD:L_0603_1608Metric" (at 224.79 56.388 90)
       (effects (font (size 1.27 1.27)) hide)
     )
@@
       (project "PicoGUS"
         (path "/8fb4b197-630e-4faa-9892-8ecaeb71c13b"
-          (reference "L1") (unit 1)
+          (reference "FB1") (unit 1)
         )
       )
@@
   (symbol (lib_id "Device:FerriteBead") (at 232.41 44.45 90) (unit 1)
     (in_bom yes) (on_board yes) (dnp no)
-    (property "Reference" "L2" (at 232.41 38.1 90)
+    (property "Reference" "FB2" (at 232.41 38.1 90)
       (effects (font (size 1.27 1.27)))
     )
@@
       (effects (font (size 1.27 1.27)))
     )
-    (property "Footprint" "Inductor_SMD:L_0402_1005Metric" (at 232.41 46.228 90)
+    (property "Footprint" "Inductor_SMD:L_0603_1608Metric" (at 232.41 46.228 90)
       (effects (font (size 1.27 1.27)) hide)
     )
@@
       (project "PicoGUS"
         (path "/8fb4b197-630e-4faa-9892-8ecaeb71c13b"
-          (reference "L2") (unit 1)
-        )
-      )
+          (reference "FB2") (unit 1)
+        )
+      )
