File: hw-hand386/PicoGUS Hand386.kicad_pcb (KiCad board)
At the start: 4 copper layers, 29.2 x 75.2 mm, 45 parts, among them J1 AudioJack3, J3 Bus_ISA_8bit, J5 AudioJack3, J6 UART_TX, U1 Pico, U10 PCM5100, U2 SN74CB3T3245, U3 SN74CB3T3257, U4 SN74CB3T3257, U5 74LVC14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

Commit message: Update Hand386 hw design
Parts:
- added REF**: OSHW-Logo_5.7x6mm_SilkScreen, Symbol:OSHW-Logo_5.7x6mm_SilkScreen, F.Cu at (123.1, 61.6)
- J3: footprint Connector_PinSocket_2.00mm:PinSocket_2x30_P2.00mm_Horizontal -> PiGUS library:EDGE-60
- moved C15 1.54 mm to (121.9, 128.6)
- moved J3 1.37 mm to (118.0, 66.0), turned to -90 degrees
- moved C2 0.42 mm to (130.6, 66.0)
Routing:
- net GND: track 73.5 -> 79.2 mm, vias 75 -> 82
- net A3: track 27.8 -> 30.0 mm
- net RESET: track 42.2 -> 44.3 mm
- net A9: track 28.0 -> 26.0 mm, vias 4 -> 3
- net A2: track 30.2 -> 28.4 mm
- net D7: track 51.3 -> 49.6 mm
- net A5: track 29.2 -> 27.6 mm, vias 2 -> 3
- net A6: track 33.3 -> 31.7 mm, vias 4 -> 5
- net A4: track 30.4 -> 28.9 mm, vias 2 -> 3
- net D3: track 52.2 -> 50.6 mm, vias 4 -> 5
- net D2: track 52.5 -> 50.9 mm, vias 4 -> 5
- net AEN: track 33.7 -> 32.2 mm, vias 2 -> 3
- net D1: track 42.9 -> 41.4 mm, vias 2 -> 3
- net D4: track 37.9 -> 36.3 mm, vias 2 -> 3
- net A7: track 31.3 -> 29.8 mm, vias 2 -> 3
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Other:
- outline, holes or cut-outs redrawn
- board text added: "Back of Hand386/Bottom of Book8088 on this side!"
- board text added: "HAND386 edition ©2023 Ian Scott"
- board text added: "HAND386 edition ©2023 Ian Scott CERN-OHL-P v2"
- board text added: "also works on BOOK8088!?"
- board text removed: "HAND386 edition ©2023 Ian Scott CERN-OHL-P"

Commit message: Prototype PicoGUS Hand386 produced on 2023-06-30
Parts:
- removed the REF** at (123.1, 61.6)
- added JP1: Jumper_2_Bridged, Connector_PinHeader_2.54mm:PinHeader_1x02_P2.54mm_Vertical, F.Cu at (124.7, 62.2)
- added JP2: SolderJumper_2_Open, Jumper:SolderJumper-2_P1.3mm_Open_RoundedPad1.0x1.5mm, B.Cu at (135.0, 127.8)
- added JP3: SolderJumper_2_Open, Jumper:SolderJumper-2_P1.3mm_Open_RoundedPad1.0x1.5mm, B.Cu at (135.0, 130.5)
- added JP4: SolderJumper_2_Open, Jumper:SolderJumper-2_P1.3mm_Open_RoundedPad1.0x1.5mm, B.Cu at (122.6, 70.1)
- added REF**: OSHW-Logo2_9.8x8mm_SilkScreen, Symbol:OSHW-Logo2_9.8x8mm_SilkScreen, B.Cu at (133.6, 121.0)
- J5: footprint PiGUS library:PJ-208-SMD -> PiGUS library:PJ-231F-4A
- U5: value 74LVC14 -> 74AHC14
- moved J5 7.17 mm to (141.0, 63.7), turned to -90 degrees
- moved R4 2.75 mm to (129.6, 63.2)
- moved FB2 2.75 mm to (132.9, 63.3)
- moved R3 2.11 mm to (129.6, 61.0)
- moved FB1 2.11 mm to (132.9, 61.1)
- moved J6 0.64 mm to (124.7, 66.0)
- turned C17 to 0 degrees
Connections:
- J3 pad 13: unconnected-(J3-UNUSED-Pad13) -> AUDIO_L_OUT
- J3 pad 15: unconnected-(J3-+12V-Pad15) -> AUDIO_R_OUT
- J3 pad 7: unconnected-(J3--5V-Pad7) -> Net-(J3--5V)
- R7 pad 1: RESET -> Net-(JP1-A)
- U5 pad 9: RESET -> Net-(JP1-A)
Routing:
- net AUDIO_R_OUT: track 0.00 -> 61.4 mm, vias 0 -> 1
- net AUDIO_L_OUT: track 0.00 -> 61.1 mm, vias 0 -> 1
- net Net-(JP1-A): track 0.00 -> 39.5 mm, vias 0 -> 2
- net RESET: track 44.3 -> 4.98 mm, vias 2 -> 0
- net Net-(FB2-Pad2): track 11.5 -> 3.73 mm
- net UART_TX: track 35.2 -> 42.5 mm
- net GND: track 79.2 -> 85.2 mm, vias 82 -> 104
- net Net-(J3--5V): track 0.00 -> 5.50 mm, vias 0 -> 1
- net D6: track 48.5 -> 46.2 mm
- net +3V3: track 38.6 -> 40.8 mm, vias 36 -> 38
- net +5V: track 79.1 -> 80.5 mm, vias 8 -> 10
- net A9: track 26.0 -> 24.9 mm
- net /Audio/AUDIO_R: track 5.83 -> 6.89 mm, vias 0 -> 1
- net Net-(FB1-Pad2): track 2.23 -> 3.25 mm
- net /Audio/AUDIO_L: track 20.4 -> 21.3 mm, vias 0 -> 1
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Other:
- board text added: "HAND386 edition ©2023 Ian Scott CERN-OHL-P v2 polpo.org/picogus"
- board text added: "RESET EN"
- board text removed: "HAND386 edition ©2023 Ian Scott CERN-OHL-P v2"

Commit message: ISA adapter v1.1/Hand386 PicoGUS v1.0
Parts:
- added JLCTOOLING1: JLCPCB-tooling, PiGUS library:JLCPCB-tooling, F.Cu at (120.6, 129.7)
- added JLCTOOLING2: JLCPCB-tooling, PiGUS library:JLCPCB-tooling, F.Cu at (127.5, 59.3)
- added JLCTOOLING3: JLCPCB-tooling, PiGUS library:JLCPCB-tooling, F.Cu at (140.7, 67.7)
- JP2, JP3, JP4: value SolderJumper_2_Open -> SolderJumper_2_Closed; footprint Jumper:SolderJumper-2_P1.3mm_Open_RoundedPad1.0x1.5mm -> Jumper:SolderJumper-2_P1.3mm_Bridged_RoundedPad1.0x1.5mm
Other:
- board text added: "v1.0"
