File: hw-hand386/PicoGUS Hand386.kicad_pcb (KiCad board)
At the start: 4 copper layers, 29.2 x 75.2 mm, 53 parts, among them J1 AudioJack3, J3 Bus_ISA_8bit, J5 AudioJack3, J6 UART_TX, U1 Pico, U10 PCM5100, U2 SN74CB3T3245, U3 SN74CB3T3257, U4 SN74CB3T3257, U5 74AHC14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

Commit message: Hand386 version and ISA adapter fabbed at JLC 8/25
Parts:
- C1, C2: footprint Capacitor_Tantalum_SMD:CP_EIA-3528-21_Kemet-B -> Capacitor_SMD:C_1206_3216Metric
- C17: footprint Capacitor_Tantalum_SMD:CP_EIA-2012-15_AVX-P -> Capacitor_SMD:C_0603_1608Metric
- D1: footprint Diode_SMD:D_SOD-123F -> Diode_SMD:D_SOD-123
- JP2, JP3, JP4: footprint Jumper:SolderJumper-2_P1.3mm_Bridged_RoundedPad1.0x1.5mm -> PiGUS library:SolderJumper-2_P1.3mm_Bridged_RoundedPad1.0x1.5mm-nomask
- moved REF** 1.47 mm to (133.6, 122.5)
- moved JLCTOOLING3 0.50 mm to (141.2, 67.7)
- moved C13 0.37 mm to (125.0, 122.5)
Routing:
- net A2: track 28.4 -> 31.3 mm
- net A3: track 30.0 -> 27.4 mm
- net DRQ: track 26.5 -> 29.1 mm
- net GND: track 85.2 -> 87.3 mm
- net D7: track 48.9 -> 50.3 mm
- net TC: track 13.6 -> 15.0 mm
- net A5: track 27.4 -> 28.7 mm
- net A6: track 31.6 -> 32.9 mm
- net A0: track 28.8 -> 27.6 mm
- net DACK: track 41.1 -> 42.2 mm
- net ~{IOW}: track 15.8 -> 16.9 mm
- net IRQ: track 20.1 -> 21.2 mm
- net D6: track 46.2 -> 47.3 mm
- net RESET: track 4.98 -> 6.05 mm
- net ~{IOR}: track 12.2 -> 13.1 mm
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Other:
- board text added: "Femto Edition ©2023 Ian Scott"
- board text added: "Femto Edition ©2023 Ian Scott CERN-OHL-P v2 polpo.org/picogus"
- board text added: "GND"
- board text added: "PICO USB vvv"
- board text added: "TX"
- board text added: "UART"
- board text added: "plugs right in to Hand386 & Book8088!"
- board text added: "v1.2"
- board text removed: "+"
- board text removed: "HAND386 edition ©2023 Ian Scott"
- board text removed: "HAND386 edition ©2023 Ian Scott CERN-OHL-P v2 polpo.org/picogus"
- board text removed: "UART TX"
- board text removed: "also works on BOOK8088!?"
- board text removed: "v1.0"

Commit message: v1.3 of Femto edition submitted to JLCPCB 2022-09-26
Parts:
- added JP5: Jumper_2_Open, Connector_PinHeader_2.54mm:PinHeader_1x02_P2.54mm_Vertical, F.Cu at (136.6, 73.7)
- moved C20 3.99 mm to (140.8, 77.7)
- moved U7 3.99 mm to (138.0, 78.2)
- moved C6 3.71 mm to (140.8, 81.3), turned to -90 degrees
- moved U9 2.99 mm to (138.1, 82.0)
- moved C1 1.93 mm to (138.7, 85.8), turned to 180 degrees
- moved REF** 0.70 mm to (133.6, 123.2)
Connections:
- U1 pad 40: unconnected-(U1-VBUS-Pad40) -> Net-(JP5-A)
Routing:
- net Net-(JP5-A): track 0.00 -> 8.44 mm
- net UART_TX: track 42.5 -> 47.2 mm
- net /VSYS: track 4.57 -> 8.83 mm
- net DACK: track 42.2 -> 38.1 mm
- net Net-(U6-Pad10): track 16.8 -> 12.9 mm, vias 2 -> 0
- net AEN: track 32.9 -> 29.1 mm
- net ~{RI/OCHRDY}: track 21.5 -> 17.8 mm
- net I/OCHRDY: track 25.4 -> 22.5 mm, vias 3 -> 1
Other:
- board text added: "Femto Edition v1.3 ©2023 Ian Scott CERN-OHL-P v2 polpo.org/picogus"
- board text removed: "Femto Edition ©2023 Ian Scott CERN-OHL-P v2 polpo.org/picogus"
- board text removed: "v1.2"
