File: hw-hand386/audio.kicad_sch (KiCad schematic)
At the start: 12 parts, among them U10 PCM5100

Commit message: Hand386 version and ISA adapter fabbed at JLC 8/25
Parts:
- C17: footprint Capacitor_Tantalum_SMD:CP_EIA-2012-15_AVX-P -> Capacitor_SMD:C_0603_1608Metric; symbol Device:C_Polarized_Small -> Device:C_Small
Changed lines of the file:
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@@
     )
   )
-  (symbol (lib_id "Device:C_Polarized_Small") (at 36.195 47.625 0) (unit 1)
+  (symbol (lib_id "Device:C_Small") (at 36.195 47.625 0) (unit 1)
     (in_bom yes) (on_board yes) (dnp no)
     (property "Reference" "C17" (at 38.735 46.355 0)
@@
       (effects (font (size 1.27 1.27)) (justify left))
     )
-    (property "Footprint" "Capacitor_Tantalum_SMD:CP_EIA-2012-15_AVX-P" (at 36.195 47.625 0)
+    (property "Footprint" "Capacitor_SMD:C_0603_1608Metric" (at 36.195 47.625 0)
       (effects (font (size 1.27 1.27)) hide)
     )
