File: hw-hand386/PicoGUS Hand386.kicad_sch (KiCad schematic)
At the start: 33 parts, among them J1 AudioJack3, J3 Bus_ISA_8bit, J5 AudioJack3, J6 UART_TX, U1 Pico, U2 SN74CB3T3245, U3 SN74CB3T3257, U4 SN74CB3T3257, U5 74LVC14, U6 74LVC00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

Commit message: Update Hand386 hw design
Parts:
- J3: footprint Connector_PinSocket_2.00mm:PinSocket_2x30_P2.00mm_Horizontal -> PiGUS library:EDGE-60
Changed lines of the file:
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@@
   )
   (symbol (lib_id "Connector:Bus_ISA_8bit") (at 46.355 62.23 0) (unit 1)
-    (in_bom yes) (on_board no) (dnp no)
+    (in_bom yes) (on_board yes) (dnp no)
     (property "Reference" "J3" (at 45.72 13.97 0)
       (effects (font (size 1.27 1.27)))
@@
       (effects (font (size 1.27 1.27)))
     )
-    (property "Footprint" "Connector_PinSocket_2.00mm:PinSocket_2x30_P2.00mm_Horizontal" (at 46.355 62.23 0)
+    (property "Footprint" "PiGUS library:EDGE-60" (at 46.355 62.23 0)
       (effects (font (size 1.27 1.27)) hide)
     )
@@
   )
   (symbol (lib_id "PiGUS library:Pico") (at 109.22 61.595 0) (unit 1)
-    (in_bom yes) (on_board no) (dnp no) (fields_autoplaced)
+    (in_bom yes) (on_board yes) (dnp no) (fields_autoplaced)
     (property "Reference" "U1" (at 109.22 29.845 0)
       (effects (font (size 1.27 1.27)))

Commit message: Prototype PicoGUS Hand386 produced on 2023-06-30
Parts:
- added JP1: Jumper_2_Bridged, Connector_PinHeader_2.54mm:PinHeader_1x02_P2.54mm_Vertical, symbol Jumper:Jumper_2_Bridged
- added JP2, JP3, JP4: SolderJumper_2_Open, Jumper:SolderJumper-2_P1.3mm_Open_RoundedPad1.0x1.5mm, symbol Jumper:SolderJumper_2_Open
- J5: footprint PiGUS library:PJ-208-SMD -> PiGUS library:PJ-231F-4A
- U5: value 74LVC14 -> 74AHC14
Connections:
- net Audio/AUDIO_L: now also JP2.2 (B)
- net Audio/AUDIO_R: now also JP3.2 (B)
- net RESET: now also JP1.2 (B); no longer R7.1, U5.9
- net UART_TX: now also JP4.2 (B)
- net AUDIO_L_OUT: now reaches J3.13 (UNUSED)
- net AUDIO_L_OUT: now also JP2.1 (A)
- net AUDIO_R_OUT: now reaches J3.15 (+12V)
- net AUDIO_R_OUT: now also JP3.1 (A)
- net at J3.7 (-5V): now also JP4.1 (A)
- new net: JP1.1 (A), R7.1, U5.9
Other:
- moved on the sheet: J1

Commit message: ISA adapter v1.1/Hand386 PicoGUS v1.0
Parts:
- JP2, JP3, JP4: value SolderJumper_2_Open -> SolderJumper_2_Closed; footprint Jumper:SolderJumper-2_P1.3mm_Open_RoundedPad1.0x1.5mm -> Jumper:SolderJumper-2_P1.3mm_Bridged_RoundedPad1.0x1.5mm; symbol Jumper:SolderJumper_2_Open -> Jumper:SolderJumper_2_Bridged
Changed lines of the file:
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@@
     )
   )
-  (symbol (lib_id "Jumper:SolderJumper_2_Open") (at 24.765 34.29 180) (unit 1)
+  (symbol (lib_id "Jumper:SolderJumper_2_Bridged") (at 24.765 34.29 180) (unit 1)
     (in_bom yes) (on_board yes) (dnp no)
     (property "Reference" "JP4" (at 24.13 40.005 90)
       (effects (font (size 1.27 1.27)) (justify right))
     )
-    (property "Value" "SolderJumper_2_Open" (at 26.035 57.15 90)
+    (property "Value" "SolderJumper_2_Closed" (at 26.035 57.15 90)
       (effects (font (size 1.27 1.27)) (justify right))
     )
-    (property "Footprint" "Jumper:SolderJumper-2_P1.3mm_Open_RoundedPad1.0x1.5mm" (at 24.765 34.29 0)
+    (property "Footprint" "Jumper:SolderJumper-2_P1.3mm_Bridged_RoundedPad1.0x1.5mm" (at 24.765 34.29 0)
       (effects (font (size 1.27 1.27)) hide)
     )
@@
     )
   )
-  (symbol (lib_id "Jumper:SolderJumper_2_Open") (at 247.015 86.36 90) (unit 1)
+  (symbol (lib_id "Jumper:SolderJumper_2_Bridged") (at 247.015 86.36 90) (unit 1)
     (in_bom yes) (on_board yes) (dnp no)
     (property "Reference" "JP2" (at 241.3 85.725 90)
       (effects (font (size 1.27 1.27)) (justify right))
     )
-    (property "Value" "SolderJumper_2_Open" (at 224.155 87.63 90)
+    (property "Value" "SolderJumper_2_Closed" (at 224.155 87.63 90)
       (effects (font (size 1.27 1.27)) (justify right))
     )
-    (property "Footprint" "Jumper:SolderJumper-2_P1.3mm_Open_RoundedPad1.0x1.5mm" (at 247.015 86.36 0)
+    (property "Footprint" "Jumper:SolderJumper-2_P1.3mm_Bridged_RoundedPad1.0x1.5mm" (at 247.015 86.36 0)
       (effects (font (size 1.27 1.27)) hide)
     )
@@
     )
   )
-  (symbol (lib_id "Jumper:SolderJumper_2_Open") (at 251.46 86.36 90) (unit 1)
+  (symbol (lib_id "Jumper:SolderJumper_2_Bridged") (at 251.46 86.36 90) (unit 1)
     (in_bom yes) (on_board yes) (dnp no)
     (property "Reference" "JP3" (at 253.365 85.725 90)
       (effects (font (size 1.27 1.27)) (justify right))
     )
-    (property "Value" "SolderJumper_2_Open" (at 253.365 87.63 90)
+    (property "Value" "SolderJumper_2_Closed" (at 253.365 87.63 90)
       (effects (font (size 1.27 1.27)) (justify right))
     )
-    (property "Footprint" "Jumper:SolderJumper-2_P1.3mm_Open_RoundedPad1.0x1.5mm" (at 251.46 86.36 0)
-      (effects (font (size 1.27 1.27)) hide)
-    )
+    (property "Footprint" "Jumper:SolderJumper-2_P1.3mm_Bridged_RoundedPad1.0x1.5mm" (at 251.46 86.36 0)
+      (effects (font (size 1.27 1.27)) hide)
+    )

Commit message: Hand386 version and ISA adapter fabbed at JLC 8/25
Parts:
- C1, C2: footprint Capacitor_Tantalum_SMD:CP_EIA-3528-21_Kemet-B -> Capacitor_SMD:C_1206_3216Metric; symbol Device:C_Polarized_US -> Device:C
- D1: footprint Diode_SMD:D_SOD-123F -> Diode_SMD:D_SOD-123
- JP2, JP3, JP4: footprint Jumper:SolderJumper-2_P1.3mm_Bridged_RoundedPad1.0x1.5mm -> PiGUS library:SolderJumper-2_P1.3mm_Bridged_RoundedPad1.0x1.5mm-nomask
Changed lines of the file:
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@@
       (effects (font (size 1.27 1.27)) (justify right))
     )
-    (property "Footprint" "Jumper:SolderJumper-2_P1.3mm_Bridged_RoundedPad1.0x1.5mm" (at 24.765 34.29 0)
+    (property "Footprint" "PiGUS library:SolderJumper-2_P1.3mm_Bridged_RoundedPad1.0x1.5mm-nomask" (at 24.765 34.29 0)
       (effects (font (size 1.27 1.27)) hide)
     )
@@
       (effects (font (size 1.27 1.27)) (justify right))
     )
-    (property "Footprint" "Jumper:SolderJumper-2_P1.3mm_Bridged_RoundedPad1.0x1.5mm" (at 247.015 86.36 0)
+    (property "Footprint" "PiGUS library:SolderJumper-2_P1.3mm_Bridged_RoundedPad1.0x1.5mm-nomask" (at 247.015 86.36 0)
       (effects (font (size 1.27 1.27)) hide)
     )
@@
       (effects (font (size 1.27 1.27)))
     )
-    (property "Footprint" "Diode_SMD:D_SOD-123F" (at 137.16 40.005 0)
+    (property "Footprint" "Diode_SMD:D_SOD-123" (at 137.16 40.005 0)
       (effects (font (size 1.27 1.27)) hide)
     )
@@
     )
   )
-  (symbol (lib_id "Device:C_Polarized_US") (at 73.66 186.69 0) (unit 1)
+  (symbol (lib_id "Device:C") (at 73.66 186.69 0) (unit 1)
     (in_bom yes) (on_board yes) (dnp no)
     (property "Reference" "C1" (at 73.66 184.15 0)
@@
       (effects (font (size 1.27 1.27)) (justify left))
     )
-    (property "Footprint" "Capacitor_Tantalum_SMD:CP_EIA-3528-21_Kemet-B" (at 73.66 186.69 0)
+    (property "Footprint" "Capacitor_SMD:C_1206_3216Metric" (at 74.6252 190.5 0)
       (effects (font (size 1.27 1.27)) hide)
     )
@@
       (effects (font (size 1.27 1.27)) (justify right))
     )
-    (property "Footprint" "Jumper:SolderJumper-2_P1.3mm_Bridged_RoundedPad1.0x1.5mm" (at 251.46 86.36 0)
+    (property "Footprint" "PiGUS library:SolderJumper-2_P1.3mm_Bridged_RoundedPad1.0x1.5mm-nomask" (at 251.46 86.36 0)
       (effects (font (size 1.27 1.27)) hide)
     )
@@
     )
   )
-  (symbol (lib_id "Device:C_Polarized_US") (at 20.955 186.69 0) (unit 1)
+  (symbol (lib_id "Device:C") (at 20.955 186.69 0) (unit 1)
     (in_bom yes) (on_board yes) (dnp no)
     (property "Reference" "C2" (at 19.685 184.785 0)
@@
       (effects (font (size 1.27 1.27)) (justify left))
     )
-    (property "Footprint" "Capacitor_Tantalum_SMD:CP_EIA-3528-21_Kemet-B" (at 20.955 186.69 0)
-      (effects (font (size 1.27 1.27)) hide)
-    )
+    (property "Footprint" "Capacitor_SMD:C_1206_3216Metric" (at 21.9202 190.5 0)
+      (effects (font (size 1.27 1.27)) hide)
+    )

Commit message: v1.3 of Femto edition submitted to JLCPCB 2022-09-26
Parts:
- added JP5: Jumper_2_Open, Connector_PinHeader_2.54mm:PinHeader_1x02_P2.54mm_Vertical, symbol Jumper:Jumper_2_Open
Connections:
- net VSYS: now also JP5.2 (B)
- net at U1.40 (VBUS): now also JP5.1 (A)
- no-connect marks 6 -> 5
Changed lines of the file:
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@@
   (junction (at 62.865 182.88) (diameter 0) (color 0 0 0 0)
   )
+  (junction (at 133.35 40.005) (diameter 0) (color 0 0 0 0)
+  )
   (junction (at 217.805 160.655) (diameter 0) (color 0 0 0 0)
   )
@@
   (junction (at 89.535 166.37) (diameter 0) (color 0 0 0 0)
   )
-  (junction (at 128.27 40.005) (diameter 0) (color 0 0 0 0)
-  )
   (junction (at 233.68 153.035) (diameter 0) (color 0 0 0 0)
   )
@@
   )
   (junction (at 47.625 190.5) (diameter 0) (color 0 0 0 0)
+  )
+  (junction (at 133.35 35.56) (diameter 0) (color 0 0 0 0)
   )
   (junction (at 67.945 190.5) (diameter 0) (color 0 0 0 0)
@@
   (no_connect (at 145.415 121.285))
   (no_connect (at 127 50.165))
-  (no_connect (at 127 37.465))
   (no_connect (at 127 45.085))
   (no_connect (at 145.415 136.525))
@@
     (stroke (width 0) (type default))
   )
-  (wire (pts (xy 128.27 40.005) (xy 127 40.005))
+  (wire (pts (xy 127 40.005) (xy 133.35 40.005))
     (stroke (width 0) (type default))
   )
@@
     (stroke (width 0) (type default))
   )
-  (wire (pts (xy 128.27 35.56) (xy 128.27 40.005))
+  (wire (pts (xy 133.35 27.305) (xy 133.35 35.56))
     (stroke (width 0) (type default))
   )
@@
     (stroke (width 0) (type default))
   )
+  (wire (pts (xy 133.35 27.305) (xy 127 27.305))
+    (stroke (width 0) (type default))
+  )
   (wire (pts (xy 175.26 88.265) (xy 175.26 93.345))
     (stroke (width 0) (type default))
@@
     (stroke (width 0) (type default))
   )
-  (wire (pts (xy 133.35 40.005) (xy 128.27 40.005))
-    (stroke (width 0) (type default))
-  )
   (wire (pts (xy 21.59 100.33) (xy 28.575 100.33))
     (stroke (width 0) (type default))
@@
   )
   (wire (pts (xy 180.34 129.54) (xy 189.23 129.54))
+    (stroke (width 0) (type default))
+  )
+  (wire (pts (xy 133.35 35.56) (xy 133.35 40.005))
     (stroke (width 0) (type default))
   )
@@
     (effects (font (size 2 2)) (justify left bottom))
   )
-  (label "VSYS" (at 129.54 40.005 0) (fields_autoplaced)
+  (label "VSYS" (at 127.635 40.005 0) (fields_autoplaced)
     (effects (font (size 1.27 1.27)) (justify left bottom))
   )
@@
     )
   )
+  (symbol (lib_id "Jumper:Jumper_2_Open") (at 127 32.385 90) (unit 1)
+    (in_bom yes) (on_board yes) (dnp no)
+    (property "Reference" "JP5" (at 128.27 31.115 90)
+      (effects (font (size 1.27 1.27)) (justify right))
+    )
+    (property "Value" "Jumper_2_Open" (at 128.27 33.655 90)
+      (effects (font (size 1.27 1.27)) (justify right))
+    )
+    (property "Footprint" "Connector_PinHeader_2.54mm:PinHeader_1x02_P2.54mm_Vertical" (at 127 32.385 0)
+      (effects (font (size 1.27 1.27)) hide)
+    )
+    (property "Datasheet" "~" (at 127 32.385 0)
+      (effects (font (size 1.27 1.27)) hide)
+    )
+    (pin "1")
+    (pin "2")
+    (instances
+      (project "PicoGUS Hand386"
+        (path "/8fb4b197-630e-4faa-9892-8ecaeb71c13b"
+          (reference "JP5") (unit 1)
+        )
+      )
+    )
+  )
   (symbol (lib_id "Device:D_Schottky") (at 137.16 40.005 0) (unit 1)
     (in_bom yes) (on_board yes) (dnp no)
@@
     )
   )
-  (symbol (lib_id "power:PWR_FLAG") (at 128.27 35.56 0) (unit 1)
+  (symbol (lib_id "power:PWR_FLAG") (at 133.35 35.56 270) (unit 1)
     (in_bom yes) (on_board yes) (dnp no) (fields_autoplaced)
-    (property "Reference" "#FLG0101" (at 128.27 33.655 0)
-      (effects (font (size 1.27 1.27)) hide)
-    )
-    (property "Value" "PWR_FLAG" (at 128.27 29.845 0)
-      (effects (font (size 1.27 1.27)))
-    )
-    (property "Footprint" "" (at 128.27 35.56 0)
-      (effects (font (size 1.27 1.27)) hide)
-    )
-    (property "Datasheet" "~" (at 128.27 35.56 0)
-      (effects (font (size 1.27 1.27)) hide)
-    )
+    (property "Reference" "#FLG0101" (at 135.255 35.56 0)
+      (effects (font (size 1.27 1.27)) hide)
+    )
+    (property "Value" "PWR_FLAG" (at 137.16 35.56 90)
+      (effects (font (size 1.27 1.27)) (justify left))
+    )
+    (property "Footprint" "" (at 133.35 35.56 0)
+      (effects (font (size 1.27 1.27)) hide)
+    )
+    (property "Datasheet" "~" (at 133.35 35.56 0)
+      (effects (font (size 1.27 1.27)) hide)
+    )
