File: hw-chipdown/RP2040.kicad_sch (KiCad schematic)
At the start: 21 parts

Commit message: Almost final PicoGUS 2.0
Parts:
- C? (x2): footprint Capacitor_SMD:C_0402_1005Metric -> Capacitor_SMD:C_0603_1608Metric
Changed lines of the file:
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@@
       (effects (font (size 1.27 1.27)) (justify left))
     )
-    (property "Footprint" "Capacitor_SMD:C_0402_1005Metric" (at 33.02 85.4202 0)
+    (property "Footprint" "Capacitor_SMD:C_0603_1608Metric" (at 33.02 85.4202 0)
       (effects (font (size 1.27 1.27)) hide)
     )
@@
       (effects (font (size 1.27 1.27)) (justify left))
     )
-    (property "Footprint" "Capacitor_SMD:C_0402_1005Metric" (at 33.02 95.5802 0)
+    (property "Footprint" "Capacitor_SMD:C_0603_1608Metric" (at 33.02 95.5802 0)
       (effects (font (size 1.27 1.27)) hide)
     )
